Commit message: testing this commit

File: src/robot/models/actuatorBot/actuator.urdf (robot description, URDF)
Before this commit: robot origins, 11 links, 9 joints
Links:
- added link middle; collision box size=0.12 0.04 0.01; visual mesh filename=model://actuatorBot/meshes/middle.dae
- link arml1: geometry collision box size=0.005 0.05 0.003; visual mesh filename=model://actuatorBot/meshes/arm1.dae
- link arml2: geometry collision box size=0.005 0.05 0.003; visual mesh filename=model://actuatorBot/meshes/arm1.dae
- link arml3: geometry collision box size=0.005 0.05 0.003; visual mesh filename=model://actuatorBot/meshes/arm1.dae
- link arml4: geometry collision box size=0.005 0.05 0.003; visual mesh filename=model://actuatorBot/meshes/arm1.dae
- link armr1: geometry collision box size=0.005 0.05 0.003; visual mesh filename=model://actuatorBot/meshes/arm1.dae
- link armr2: geometry collision box size=0.005 0.05 0.003; visual mesh filename=model://actuatorBot/meshes/arm1.dae
- link armr3: geometry collision box size=0.005 0.05 0.003; visual mesh filename=model://actuatorBot/meshes/arm1.dae
- link armr4: geometry collision box size=0.005 0.05 0.003; visual mesh filename=model://actuatorBot/meshes/arm1.dae
- link base_link: mass None -> 1.0; geometry collision box size=0.13 0.25 0.005; visual mesh filename=model://actuatorBot/meshes/base.dae
- link carriage1: geometry collision box size=0.12 0.03 0.015; visual mesh filename=model://actuatorBot/meshes/carriage.dae
- link carriage2: geometry collision box size=0.12 0.03 0.015; visual mesh filename=model://actuatorBot/meshes/carriage.dae
Joints:
- removed joint carriage1 to arml2
- removed joint carriage1 to armr2
- removed joint carriage2 to arml3
- added joint carriage1 to arml3: type fixed, parent carriage1, child arml3, origin xyz=0.0625 -0.09 0
- added joint carriage1 to armr3: type fixed, parent carriage1, child armr3, origin xyz=-0.0625 -0.09 0
- added joint carriage2 to arml2: type fixed, parent carriage2, child arml2, origin xyz=0.0625 0.105 0
- added joint carriage2 to armr2: type fixed, parent carriage2, child armr2, origin xyz=-0.0625 0.105 0
- added joint middleStuff: type fixed, parent base_link, child middle, origin xyz=0 0 0.0125
- joint base_to_carriage1: origin xyz=0 -0.05 0.01 -> xyz=0 0.06 0.0125
- joint base_to_carriage2: origin xyz=0 0.05 0.01 -> xyz=0 -0.06 0.0125
- joint carriage1 to arml1: origin xyz=0.06 -0.005 0 -> xyz=0.0625 -0.105 0
- joint carriage1 to armr1: origin xyz=-0.06 -0.005 0 -> xyz=-0.0625 -0.105 0
- joint carriage2 to arml4: origin xyz=0.06 0.005 0 -> xyz=0.0625 0.09 0
- joint carriage2 to armr4: child armr2 -> armr4; origin xyz=-0.06 0.005 0 -> xyz=-0.0625 0.09 0

Commit message: Editting URDF and adding in Moveit Configurations

File: src/robot/models/actuatorBot/actuator.urdf (robot description, URDF)
Before this commit: robot origins, 12 links, 11 joints
Links:
- link arml1: mass None -> 1.0
- link arml2: mass None -> 1.0
- link arml3: mass None -> 1.0
- link arml4: mass None -> 1.0
- link armr1: mass None -> 1.0
- link armr2: mass None -> 1.0
- link armr3: mass None -> 1.0
- link armr4: mass None -> 1.0
- link base_link: geometry collision box size=0.13 0.25 0.0075; visual mesh filename=model://actuatorBot/meshes/base.dae
- link carriage1: mass None -> 1.0
- link carriage2: mass None -> 1.0
- link middle: mass None -> 1.0; geometry collision box size=0.12 0.06 0.01; visual mesh filename=model://actuatorBot/meshes/middle1.dae
Joints:
- removed joint middleStuff
- added joint arml1 to middle: type continuous, parent arml1, child middle, origin xyz=-0.0625 -0.045 0 rpy=0.7853981625 0 0, axis 1 0 0
- joint base_to_carriage1: axis (none) -> 0 1 0; limit (none) -> lower=-0.08 upper=.08 effort=1000.0 velocity=0.5; origin xyz=0 0.06 0.0125 -> xyz=0 0.045 0.0075; type fixed -> prismatic
- joint base_to_carriage2: axis (none) -> 0 1 0; limit (none) -> lower=-0.08 upper=0.08 effort=1000.0 velocity=0.5; origin xyz=0 -0.06 0.0125 -> xyz=0 -0.045 0.0075; type fixed -> prismatic
- joint carriage1 to arml1: axis (none) -> 1 0 0; origin xyz=0.0625 -0.105 0 -> xyz=0.0625 0.008 0 rpy=-0.7853981625 0 0; type fixed -> continuous
- joint carriage1 to arml3: axis (none) -> 1 0 0; origin xyz=0.0625 -0.09 0 -> xyz=0.0625 -0.008 0 rpy=-0.7853981625 0 0; type fixed -> continuous
- joint carriage1 to armr1: axis (none) -> 1 0 0; origin xyz=-0.0625 -0.105 0 -> xyz=-0.0625 0.008 0 rpy=-0.7853981625 0 0; type fixed -> continuous
- joint carriage1 to armr3: axis (none) -> 1 0 0; origin xyz=-0.0625 -0.09 0 -> xyz=-0.0625 -0.008 0 rpy=-0.7853981625 0 0; type fixed -> continuous
- joint carriage2 to arml2: axis (none) -> 1 0 0; origin xyz=0.0625 0.105 0 -> xyz=0.0625 0.008 0 rpy=0.7853981625 0 0; type fixed -> continuous
- joint carriage2 to arml4: axis (none) -> 1 0 0; origin xyz=0.0625 0.09 0 -> xyz=0.0625 -0.008 0 rpy=0.7853981625 0 0; type fixed -> continuous
- joint carriage2 to armr2: axis (none) -> 1 0 0; origin xyz=-0.0625 0.105 0 -> xyz=-0.0625 -0.008 0 rpy=0.7853981625 0 0; type fixed -> continuous
- joint carriage2 to armr4: axis (none) -> 1 0 0; origin xyz=-0.0625 0.09 0 -> xyz=-0.0625 0.008 0 rpy=0.7853981625 0 0; type fixed -> continuous
